Commit message: vision improved

File: ros2_iiwa/iiwa_description/urdf/iiwa.urdf.xacro (robot description, xacro)
@@ -251,4 +251,10 @@
     <origin xyz="0.0 0 0.0" rpy="3.14 -1.57 0"/>
   </joint>
+  <link name="${prefix}camera_link_optical"/>
+<joint name="${prefix}camera_optical_joint" type="fixed">
+  <parent link="${prefix}camera_link"/>
+  <child link="${prefix}camera_link_optical"/>
+  <origin xyz="0 0 0" rpy="-1.5708 0 -1.5708"/>
+</joint>
 <gazebo reference="${prefix}camera_link">
   <sensor name="camera" type="camera">
