Commit message: navigation completed

File: ros2_fra2mo/urdf/fra2mo_base_macro.xacro (robot description, xacro)
@@ -121,4 +121,81 @@
       <origin xyz="0.0 0.0 0.125" rpy="0 0 0" />
     </joint>
+    <joint name="lidar_basket_joint" type="fixed">
+      <parent link="lidar_link" />
+      <child link="basket_link" />
+      <origin xyz="0.0 0.0 0.05" rpy="0 0 0" />
+    </joint>
+   <link name="basket_link">
+  <visual>
+    <origin xyz="0 0 0" rpy="0 0 0" />
+    <geometry>
+      <box size="0.25 0.25 0.02" />
+    </geometry>
+    <material name="White"><color rgba="1 1 1 1"/></material>
+  </visual>
+  <collision>
+    <origin xyz="0 0 0" rpy="0 0 0" />
+    <geometry>
+      <box size="0.25 0.25 0.02" />
+    </geometry>
+  </collision>
+  <visual>
+    <origin xyz="0.125 0 0.06" rpy="0 0 0" />
+    <geometry>
+      <box size="0.02 0.25 0.12" />
+    </geometry>
+    <material name="White"><color rgba="1 1 1 1"/></material>
+  </visual>
+  <collision>
+    <origin xyz="0.15 0 0.05" rpy="0 0 0" />
+    <geometry>
+      <box size="0.02 0.3 0.1" />
+    </geometry>
+  </collision>
+  <visual>
+    <origin xyz="0.0 0.125 0.06" rpy="0 0 0" />
+    <geometry>
+      <box size="0.25 0.02 0.12" />
+    </geometry>
+    <material name="White"><color rgba="1 1 1 1"/></material>
+  </visual>
+  <collision>
+    <origin xyz="0.0 0.125 0.06" rpy="0 0 0" />
+    <geometry>
+      <box size="0.25 0.02 0.12" />
+    </geometry>
+  </collision>
+  <visual>
+    <origin xyz="-0.125 0 0.06" rpy="0 0 0" />
+    <geometry>
+      <box size="0.02 0.25 0.12" />
+    </geometry>
+    <material name="White"><color rgba="1 1 1 1"/></material>
+  </visual>
+  <collision>
+    <origin xyz="-0.125 0 0.06" rpy="0 0 0" />
+    <geometry>
+      <box size="0.02 0.25 0.12" />
+    </geometry>
+  </collision>
+  <visual>
+    <origin xyz="0.0 -0.125 0.06" rpy="0 0 0" />
+    <geometry>
+      <box size="0.25 0.02 0.12" />
+    </geometry>
+    <material name="White"><color rgba="1 1 1 1"/></material>
+  </visual>
+  <collision>
+    <origin xyz="0.0 -0.125 0.06" rpy="0 0 0" />
+    <geometry>
+      <box size="0.25 0.02 0.12" />
+    </geometry>
+  </collision>
+  <inertial>
+    <origin xyz="0 0 0" />
+    <mass value="0.1" />
+    <inertia ixx="0.001" ixy="0.0" ixz="0.0" iyy="0.001" iyz="0.0" izz="0.001" />
+  </inertial>
+</link>
     <!-- Gazebo Material Assignments
     <gazebo reference="base_link">

File: ros2_iiwa/iiwa_description/urdf/iiwa.urdf.xacro (robot description, xacro)
@@ -235,4 +235,5 @@
       </material>
     </visual>
+    <!--
     <collision>
       <geometry>
@@ -240,4 +241,5 @@
       </geometry>
     </collision>
+    -->
     <inertial>
       <mass value="0.1" />
